File: PCB/CyberDock.kicad_pcb (KiCad board)
At the start: 2 copper layers, 82 x 79.6 mm, 26 parts, among them SW1 SW_Push_45deg, SW10 SW_Push_45deg, SW11 SW_Push_45deg, SW12 SW_Push_45deg, SW2 SW_Push_45deg, SW3 SW_Push_45deg, SW5 SW_Push_45deg, SW6 SW_Push_45deg, SW7 SW_Push_45deg, SW8 SW_Push_45deg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

Commit message: Add files via upload
Routing:
- net GND: track 44.3 -> 72.7 mm
- added copper zone on B.Cu, net GND
- added copper zone on F.Cu, net GND
Changed lines of the file:
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@@
+	)
+	(segment
+		(start 160.133 57.407)
+		(end 172.133 57.407)
+		(width 0.5)
+		(layer "F.Cu")
+		(net 1)
+	)
+	(segment
+		(start 172.133 57.407)
+		(end 183.62 45.92)
+		(width 0.5)
+		(layer "F.Cu")
+		(net 1)
+	)
+	(segment
+		(start 160 57.54)
+		(end 160.133 57.407)
+		(width 0.5)
+		(layer "F.Cu")
+		(net 1)
 	)
 	(segment
@@
 	)
 	(segment
+		(start 118 59)
+		(end 139.725 59)
+		(width 0.5)
+		(layer "F.Cu")
+		(net 4)
+	)
+	(segment
 		(start 114.3 80.01875)
 		(end 171.44125 80.01875)
@@
 	)
 	(segment
+		(start 150.265 48.46)
+		(end 168.38 48.46)
+		(width 0.5)
+		(layer "F.Cu")
+		(net 4)
+	)
+	(segment
 		(start 114.3 80.01875)
 		(end 113.049 78.76775)
@@
 	)
 	(segment
+		(start 139.725 59)
+		(end 150.265 48.46)
+		(width 0.5)
+		(layer "F.Cu")
+		(net 4)
+	)
+	(segment
+		(start 113.049 63.951)
+		(end 118 59)
+		(width 0.5)
+		(layer "F.Cu")
+		(net 4)
+	)
+	(segment
+		(start 171.44125 80.01875)
+		(end 171.45 80.01)
+		(width 0.5)
+		(layer "F.Cu")
+		(net 4)
+	)
+	(segment
 		(start 113.049 78.76775)
 		(end 113.049 63.951)
@@
 	)
 	(segment
-		(start 118 59)
-		(end 139 59)
-		(width 0.5)
-		(layer "F.Cu")
-		(net 4)
-	)
-	(segment
-		(start 149.54 48.46)
-		(end 168.38 48.46)
-		(width 0.5)
-		(layer "F.Cu")
-		(net 4)
-	)
-	(segment
-		(start 171.44125 80.01875)
-		(end 171.45 80.01)
-		(width 0.5)
-		(layer "F.Cu")
-		(net 4)
-	)
-	(segment
-		(start 113.049 63.951)
-		(end 118 59)
-		(width 0.5)
-		(layer "F.Cu")
-		(net 4)
-	)
-	(segment
-		(start 139 59)
-		(end 149.54 48.46)
-		(width 0.5)
-		(layer "F.Cu")
-		(net 4)
-	)
-	(segment
 		(start 136.8425 68.8975)
 		(end 133.35 72.39)
@@
 	)
 	(segment
-		(start 139 58)
-		(end 151.08 45.92)
-		(width 0.5)
-		(layer "F.Cu")
-		(net 9)
-	)
-	(segment
-		(start 151.08 45.92)
-		(end 168.38 45.92)
-		(width 0.5)
-		(layer "F.Cu")
-		(net 9)
-	)
-	(segment
-		(start 118.008636 58)
-		(end 139 58)
-		(width 0.5)
-		(layer "F.Cu")
-		(net 9)
-	)
-	(segment
 		(start 112.348 97.108)
 		(end 112.348 63.660636)
@@
 	)
 	(segment
+		(start 118.008636 58)
+		(end 139.6 58)
+		(width 0.5)
+		(layer "F.Cu")
+		(net 9)
+	)
+	(segment
+		(start 151.68 45.92)
+		(end 168.38 45.92)
+		(width 0.5)
+		(layer "F.Cu")
+		(net 9)
+	)
+	(segment
+		(start 114.3 99.06)
+		(end 112.348 97.108)
+		(width 0.5)
+		(layer "F.Cu")
+		(net 9)
+	)
+	(segment
+		(start 112.348 63.660636)
+		(end 118.008636 58)
+		(width 0.5)
+		(layer "F.Cu")
+		(net 9)
+	)
+	(segment
+		(start 139.6 58)
+		(end 151.68 45.92)
+		(width 0.5)
+		(layer "F.Cu")
+		(net 9)
+	)
+	(segment
 		(start 114.3 99.06)
 		(end 171.45 99.06)
@@
 	)
 	(segment
-		(start 114.3 99.06)
-		(end 112.348 97.108)
-		(width 0.5)
-		(layer "F.Cu")
-		(net 9)
-	)
-	(segment
-		(start 112.348 63.660636)
-		(end 118.008636 58)
-		(width 0.5)
-		(layer "F.Cu")
-		(net 9)
-	)
-	(segment
 		(start 136.8425 87.9475)
 		(end 133.35 91.44)
@@
 	)
 	(segment
+		(start 118.017272 57)
+		(end 139.475 57)
+		(width 0.5)
+		(layer "F.Cu")
+		(net 14)
+	)
+	(segment
+		(start 111.647 115.457)
+		(end 111.647 63.370272)
+		(width 0.5)
+		(layer "F.Cu")
+		(net 14)
+	)
+	(segment
+		(start 153.095 43.38)
+		(end 168.38 43.38)
+		(width 0.5)
+		(layer "F.Cu")
+		(net 14)
+	)
+	(segment
+		(start 114.3 118.11)
+		(end 171.45 118.11)
+		(width 0.5)
+		(layer "F.Cu")
+		(net 14)
+	)
+	(segment
 		(start 114.3 118.11)
 		(end 111.647 115.457)
@@
 	)
 	(segment
-		(start 139.008636 57)
-		(end 152.628636 43.38)
-		(width 0.5)
-		(layer "F.Cu")
-		(net 14)
-	)
-	(segment
-		(start 114.3 118.11)
-		(end 171.45 118.11)
-		(width 0.5)
-		(layer "F.Cu")
-		(net 14)
-	)
-	(segment
-		(start 118.017272 57)
-		(end 139.008636 57)
-		(width 0.5)
-		(layer "F.Cu")
-		(net 14)
-	)
-	(segment
-		(start 111.647 115.457)
-		(end 111.647 63.370272)
-		(width 0.5)
-		(layer "F.Cu")
-		(net 14)
-	)
-	(segment
-		(start 152.628636 43.38)
-		(end 168.38 43.38)
+		(start 139.475 57)
+		(end 153.095 43.38)
 		(width 0.5)
 		(layer "F.Cu")
@@
 		(net 25)
 	)
+	(zone
+		(net 1)
+		(net_name "GND")
+		(layers "F.Cu" "B.Cu")
+		(hatch edge 0.5)
+		(connect_pads
+			(clearance 0.5)
+		)
+		(min_thickness 0.25)
+		(filled_areas_thickness no)
+		(fill yes
+			(thermal_gap 0.5)
+			(thermal_bridge_width 0.5)
+		)
+		(polygon
+			(pts
+				(xy 191.5 40.475) (xy 191.5 120.05) (xy 109.55 120.05) (xy 109.55 64.3) (xy 119.075 54.775) (xy 140.5 54.775)
+				(xy 154.8 40.475)
+			)
+		)
+	)
 	(embedded_fonts no)
